Commit message: Add files via upload

File: mobile_description/urdf/mobile.xacro (robot description, xacro)
@@ -215,4 +215,30 @@
 <axis xyz="1 0 0"/>
 </joint>
+ <joint name="hokuyo_joint" type="fixed">
+    <axis xyz="0 1 0" />
+    <origin xyz="0 0 0.21" rpy="0 0 0"/>
+    <parent link="base_link"/>
+    <child link="hokuyo_link"/>
+  </joint>
+  <!-- Hokuyo Laser -->
+  <link name="hokuyo_link">
+    <collision>
+      <origin xyz="0 0 0" rpy="0 0 0"/>
+      <geometry>
+    <box size="0.1 0.1 0.1"/>
+      </geometry>
+    </collision>
+    <visual>
+      <origin xyz="0 0 0" rpy="0 0 0"/>
+      <geometry>
+        <mesh filename="package://mobile_description/meshes/hokuyo.dae"/>
+      </geometry>
+    </visual>
+    <inertial>
+      <mass value="1e-5" />
+      <origin xyz="0 0 0" rpy="0 0 0"/>
+      <inertia ixx="1e-6" ixy="0" ixz="0" iyy="1e-6" iyz="0" izz="1e-6" />
+    </inertial>
+  </link>
 <transmission name="tran1">
     <type>transmission_interface/SimpleTransmission</type>

Commit message: Add files via upload

File: mobile_description/urdf/mobile.xacro (robot description, xacro)
@@ -58,5 +58,5 @@
         <origin xyz="0 0 0" rpy="0 0 0"/>
         <geometry>
-         <cylinder length="0.05" radius="0.05"/>
+         <cylinder length="0.04" radius="0.05"/>
           </geometry>
 </collision>
@@ -92,5 +92,5 @@
         <origin xyz="0 0 0" rpy="0 0 0"/>
         <geometry>
-         <cylinder length="0.05" radius="0.05"/>
+         <cylinder length="0.04" radius="0.05"/>
           </geometry>
 </collision>
@@ -126,5 +126,5 @@
         <origin xyz="0 0 0" rpy="0 0 0"/>
         <geometry>
-         <cylinder length="0.05" radius="0.05"/>
+         <cylinder length="0.04" radius="0.05"/>
           </geometry>
 </collision>
@@ -160,5 +160,5 @@
         <origin xyz="0 0 0" rpy="0 0 0"/>
         <geometry>
-         <cylinder length="0.05" radius="0.05"/>
+         <cylinder length="0.04" radius="0.05"/>
           </geometry>
 </collision>
@@ -241,4 +241,38 @@
     </inertial>
   </link>
+<link name="sonar_link">
+          <visual>
+              <origin xyz="0 0 0" rpy="0 0 0"/>
+              <geometry>
+              <sphere radius="0.01"/>
+              </geometry>
+              <material name="blue">
+              <color rgba="0 0 1 1"/>
+              </material>
+          </visual>
+      <collision>
+        <origin xyz="0 0 0" rpy="0 0 0"/>
+        <geometry>
+         <sphere radius="0.01"/>
+          </geometry>
+</collision>
+<inertial>
+   <mass
+        value="0.01" />
+      <inertia
+        ixx="0.00301717973628494"
+        ixy="-3.18755438710738E-17"
+        ixz="-6.24500451351651E-17"
+        iyy="0.0176625083227497"
+        iyz="-0.000444787144430361"
+        izz="0.015853003043962" />
+</inertial>
+</link>
+<joint name="sonar_joint" type="fixed">
+   <origin xyz="0.14 0.02 0.16" rpy="0 0 0" />
+   <parent link="base_link"/>
+   <child link="sonar_link" />
+<axis xyz="0 1 0"/>
+</joint>
 <transmission name="tran1">
     <type>transmission_interface/SimpleTransmission</type>
